Commit message: Good progress

File: urdf/robotiq_gripper.ros2_control.xacro (robot description, xacro)
@@ -4,6 +4,6 @@
         name
         prefix
+        sim_gazebo:=false
         sim_ignition:=false
-        sim_gazebo:=false
         sim_isaac:=false
         isaac_joint_commands:=/isaac_joint_commands
@@ -50,5 +50,5 @@
             </hardware>
             <!-- Joint interfaces -->
-            <!-- With Ignition or Hardware, they handle mimic joints, so we only need this command interface activated -->
+            <!-- With Ignition or Hardware, they handle  joints, so we only need this command interface activated -->
             <joint name="${prefix}robotiq_85_left_knuckle_joint">
                 <command_interface name="position" />
@@ -61,5 +61,5 @@
             <xacro:if value="${sim_gazebo or use_fake_hardware or sim_isaac or sim_ignition}">
                 <joint name="${prefix}robotiq_85_right_knuckle_joint">
-                    <param name="mimic">${prefix}robotiq_85_left_knuckle_joint</param>
+                    <param name="">${prefix}robotiq_85_left_knuckle_joint</param>
                     <param name="multiplier">-1</param>
                     <xacro:unless value="${sim_ignition}">
@@ -70,5 +70,5 @@
                 </joint>
                 <joint name="${prefix}robotiq_85_left_inner_knuckle_joint">
-                    <param name="mimic">${prefix}robotiq_85_left_knuckle_joint</param>
+                    <param name="">${prefix}robotiq_85_left_knuckle_joint</param>
                     <param name="multiplier">1</param>
                     <xacro:unless value="${sim_ignition}">
@@ -79,5 +79,5 @@
                 </joint>
                 <joint name="${prefix}robotiq_85_right_inner_knuckle_joint">
-                    <param name="mimic">${prefix}robotiq_85_left_knuckle_joint</param>
+                    <param name="">${prefix}robotiq_85_left_knuckle_joint</param>
                     <param name="multiplier">-1</param>
                     <xacro:unless value="${sim_ignition}">
@@ -88,5 +88,5 @@
                 </joint>
                 <joint name="${prefix}robotiq_85_left_finger_tip_joint">
-                    <param name="mimic">${prefix}robotiq_85_left_knuckle_joint</param>
+                    <param name="">${prefix}robotiq_85_left_knuckle_joint</param>
                     <param name="multiplier">-1</param>
                     <xacro:unless value="${sim_ignition}">
@@ -97,5 +97,5 @@
                 </joint>
                 <joint name="${prefix}robotiq_85_right_finger_tip_joint">
-                    <param name="mimic">${prefix}robotiq_85_left_knuckle_joint</param>
+                    <param name="">${prefix}robotiq_85_left_knuckle_joint</param>
                     <param name="multiplier">1</param>
                     <xacro:unless value="${sim_ignition}">

File: urdf/robotiq_gripper_macro.xacro (robot description, xacro)
@@ -6,5 +6,5 @@
         parent
         *origin
-        sim_gazebo=false
+        sim_gazebo:=false
         sim_ignition:=false
         sim_isaac:=false

File: urdf/ur5_gripper.urdf.xacro (robot description, xacro)
@@ -4,4 +4,5 @@
    <xacro:arg name="name" default="ur"/>
    <!-- import main macro -->
+   <!-- <xacro:include filename="$(find custom_ur_franka)/urdf/camera.xacro"/> -->
    <xacro:include filename="$(find custom_ur_franka)/urdf/ur5_macro.xacro"/>
    <!-- possible 'ur_type' values: ur3, ur3e, ur5, ur5e, ur7e, ur10, ur10e, ur12e, ur16e, ur15, ur20, ur30 -->
@@ -76,32 +77,4 @@
        <child link="ground_plane"/>
      </joint>
-       <!-- White table -->
-    <link name="table_link">
-      <visual>
-        <origin xyz="0 0 0.375" rpy="0 0 0"/>
-        <geometry>
-          <box size="1.5 0.8 0.05"/>  <!-- L x W x thickness -->
-        </geometry>
-        <material name="white">
-          <color rgba="1 1 1 1"/>
-        </material>
-      </visual>
-      <collision>
-        <origin xyz="0 0 0.375" rpy="0 0 0"/>
-        <geometry>
-          <box size="1.5 0.8 0.05"/>
-        </geometry>
-      </collision>
-      <inertial>
-        <mass value="5"/>
-        <origin xyz="0 0 0.375"/>
-        <inertia ixx="1" ixy="0" ixz="0" iyy="1" iyz="0" izz="1"/>
-      </inertial>
-    </link>
-    <joint name="table_joint" type="fixed">
-      <parent link="world"/>
-      <child link="table_link"/>
-      <origin xyz="0 0 0.4" rpy="0 0 0"/>  <!-- Table height is 0.4 m -->
-    </joint>
    </xacro:if>
    <!-- arm -->
@@ -143,5 +116,5 @@
      trajectory_port="$(arg trajectory_port)"
      >
-     <origin xyz="0 0 0.80" rpy="0 0 0" />          <!-- position robot in the world -->
+     <origin xyz="0 0 0.8" rpy="0 0 0" />          <!-- position robot in the world -->
    </xacro:ur_robot>
    <xacro:if value="$(arg sim_gazebo)">
@@ -166,11 +139,14 @@
     </gazebo>
   </xacro:if>
-  <!-- parameters -->
-    <xacro:arg name="use_fake_hardware" default="true" />
-    <xacro:arg name="com_port" default="/dev/ttyUSB0" />
-    <!-- Import macros -->
-    <xacro:include filename="$(find custom_ur_franka)/urdf/robotiq_gripper_macro.xacro" />
-    <xacro:robotiq_gripper name="RobotiqGripperHardwareInterface" prefix="" parent="tool0" use_fake_hardware="$(arg use_fake_hardware)" com_port="$(arg com_port)" sim_gazebo="$(arg sim_gazebo)">
-        <origin xyz="0 0 0" rpy="0 0 0" />
-    </xacro:robotiq_gripper>
+  <xacro:arg name="use_fake_hardware" default="true" />
+  <xacro:arg name="com_port" default="/dev/ttyUSB0" />
+  <!-- In your URDF/Xacro -->
+  <!-- <xacro:include filename="$(find robotiq_description)/urdf/robotiq_85_gripper.xacro"/>
+  <xacro:robotiq_85_gripper parent="ee_link" prefix="robotiq_85_" />
+ -->
+  <!-- Import macros -->
+  <xacro:include filename="$(find custom_ur_franka)/urdf/robotiq_gripper_macro.xacro" />
+  <xacro:robotiq_gripper name="RobotiqGripperHardwareInterface" prefix="" parent="tool0" use_fake_hardware="$(arg use_fake_hardware)" com_port="$(arg com_port)" sim_gazebo="$(arg sim_gazebo)">
+    <origin xyz="0 0 0" rpy="0 0 0" />
+  </xacro:robotiq_gripper>
 </robot>
