Commit message: simple changes

File: urdf/ur5_gripper.urdf.xacro (robot description, xacro)
@@ -77,4 +77,44 @@
        <child link="ground_plane"/>
      </joint>
+        <!-- White table -->
+    <link name="table_link">
+      <visual>
+        <origin xyz="0 0 0.375" rpy="0 0 0"/>
+        <geometry>
+          <box size="1.5 0.8 0.05"/>  <!-- L x W x thickness -->
+        </geometry>
+        <material name="white">
+          <color rgba="1 1 1 1"/>
+        </material>
+      </visual>
+      <collision>
+        <origin xyz="0 0 0.375" rpy="0 0 0"/>
+        <geometry>
+          <box size="1.5 0.8 0.05"/>
+        </geometry>
+      </collision>
+      <inertial>
+        <mass value="5"/>
+        <origin xyz="0 0 0.375"/>
+        <inertia ixx="1" ixy="0" ixz="0" iyy="1" iyz="0" izz="1"/>
+      </inertial>
+    </link>
+    <joint name="table_joint" type="fixed">
+      <parent link="world"/>
+      <child link="table_link"/>
+      <origin xyz="0 0 0.4" rpy="0 0 0"/>  <!-- Table height is 0.4 m -->
+    </joint>
+     <xacro:if value="${is_sim_gazebo}">
+       <gazebo reference="ground_plane">
+         <material>Gazebo/White</material>
+         <static>1</static>
+       </gazebo>
+     </xacro:if>
+     <xacro:if value="${is_sim_ignition}">
+       <ignition reference="ground_plane">
+         <material>Gazebo/White</material>
+         <static>1</static>
+       </ignition>
+     </xacro:if>
    </xacro:if>
    <!-- arm -->
